Commit message: acrungus

File: urdf/robot.urdf (robot description, URDF)
Before this commit: robot roscontrol, 4 links, 3 joints
Links:
- link box: geometry collision box size=0.08 0.08 0.08; visual box size=0.08 0.3 0.08
Joints:
- joint gripper_extension: origin xyz=${width-.01} 0 0.2 rpy=0 0 0 -> xyz=${width-.01} 0 0.1 rpy=0 0 0
- joint tobox: origin xyz=${.707*width+0.04} 0 ${.707*width} -> xyz=${.707*width+0.04} 0 ${.507*width}
